File: hardware/e-wall-smd.brd (EAGLE design)
At the start: 50.8 x 48.3 mm, 67 parts, among them IC1 74HCT595D, IC2 74HCT595D, IC3 74HCT595D, IC4 74HCT595D, Q1 2N7002P, Q10 2N7002P, Q11 2N7002P, Q12 2N7002P, Q13 2N7002P, Q14 2N7002P, Q15 2N7002P, Q16 2N7002P, Q17 2N7002P, Q18 2N7002P, Q19 2N7002P, Q2 2N7002P, Q20 2N7002P, Q21 2N7002P, Q22 2N7002P, Q23 2N7002P, Q24 2N7002P, Q25 IRF8313P, Q26 IRF8313P, Q27 IRF8313P, Q28 IRF8313P, Q3 2N7002P, Q4 2N7002P, Q5 2N7002P, Q6 2N7002P, Q7 2N7002P, Q8 2N7002P, Q9 2N7002P, T1 BC547, T2 BC557, T3 BC547

Commit message: Kleine anpassungen im Layout
Routing:
- net +5V: track 96.3 -> 97.1 mm
- net CP: vias 50 -> 48
Changed lines of the file:
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@@
 <setting verticaltext="up"/>
 </settings>
-<grid distance="10" unitdist="mil" unit="mil" style="dots" multiple="1" display="yes" altdistance="0.025" altunitdist="inch" altunit="inch"/>
+<grid distance="50" unitdist="mil" unit="mil" style="dots" multiple="1" display="yes" altdistance="0.025" altunitdist="inch" altunit="inch"/>
 <layers>
 <layer number="1" name="Top" color="4" fill="1" visible="yes" active="yes"/>
@@
 <vertex x="50.8" y="24.13"/>
 <vertex x="45.72" y="19.05"/>
-<vertex x="45.72" y="8.89"/>
-<vertex x="44.45" y="7.62"/>
-<vertex x="39.37" y="7.62"/>
-<vertex x="38.1" y="8.89"/>
+<vertex x="45.72" y="10.16"/>
+<vertex x="44.45" y="8.89"/>
+<vertex x="39.37" y="8.89"/>
+<vertex x="38.1" y="10.16"/>
 <vertex x="38.1" y="22.86"/>
 <vertex x="44.45" y="29.21"/>
@@
 <vertex x="50.8" y="24.13"/>
 <vertex x="45.72" y="19.05"/>
-<vertex x="45.72" y="8.89"/>
-<vertex x="44.45" y="7.62"/>
-<vertex x="39.37" y="7.62"/>
-<vertex x="38.1" y="8.89"/>
+<vertex x="45.72" y="10.16"/>
+<vertex x="44.45" y="8.89"/>
+<vertex x="39.37" y="8.89"/>
+<vertex x="38.1" y="10.16"/>
 <vertex x="38.1" y="22.86"/>
 <vertex x="44.45" y="29.21"/>
@@
 <via x="36.83" y="22.86" extent="1-16" drill="0.6"/>
 <via x="35.814" y="22.86" extent="1-16" drill="0.6"/>
-<via x="14.478" y="19.812" extent="1-16" drill="0.6"/>
-<via x="15.494" y="19.812" extent="1-16" drill="0.6"/>
-<via x="16.51" y="19.812" extent="1-16" drill="0.6"/>
-<via x="17.526" y="19.812" extent="1-16" drill="0.6"/>
-<via x="18.542" y="19.812" extent="1-16" drill="0.6"/>
-<via x="19.558" y="19.812" extent="1-16" drill="0.6"/>
 <via x="18.034" y="22.606" extent="1-16" drill="0.6"/>
 <via x="17.018" y="22.606" extent="1-16" drill="0.6"/>
@@
 <via x="32.004" y="35.052" extent="1-16" drill="0.6"/>
 <via x="32.512" y="35.814" extent="1-16" drill="0.6"/>
+<via x="29.718" y="6.858" extent="1-16" drill="0.6"/>
+<via x="25.654" y="6.858" extent="1-16" drill="0.6"/>
+<via x="19.304" y="6.858" extent="1-16" drill="0.6"/>
+<via x="1.27" y="21.59" extent="1-16" drill="0.6"/>
 </signal>
 <signal name="VCC" class="1">
@@
 <vertex x="45.72" y="27.94"/>
 <vertex x="39.37" y="21.59"/>
-<vertex x="39.37" y="10.16"/>
-<vertex x="40.64" y="8.89"/>
-<vertex x="43.18" y="8.89"/>
-<vertex x="44.45" y="10.16"/>
+<vertex x="39.37" y="11.43"/>
+<vertex x="40.64" y="10.16"/>
+<vertex x="43.18" y="10.16"/>
+<vertex x="44.45" y="11.43"/>
 <vertex x="44.45" y="20.32"/>
 <vertex x="50.8" y="26.67"/>
@@
 <vertex x="45.72" y="27.94"/>
 <vertex x="39.37" y="21.59"/>
-<vertex x="39.37" y="10.16"/>
-<vertex x="40.64" y="8.89"/>
-<vertex x="43.18" y="8.89"/>
-<vertex x="44.45" y="10.16"/>
+<vertex x="39.37" y="11.43"/>
+<vertex x="40.64" y="10.16"/>
+<vertex x="43.18" y="10.16"/>
+<vertex x="44.45" y="11.43"/>
 <vertex x="44.45" y="20.32"/>
 <vertex x="50.8" y="26.67"/>
@@
 <wire x1="19.812" y1="4.318" x2="20.574" y2="5.08" width="0.8128" layer="1"/>
 <contactref element="TP3" pad="TP"/>
-<wire x1="33.02" y1="5.08" x2="29.464" y2="5.08" width="0.8128" layer="16"/>
-<wire x1="29.464" y1="5.08" x2="28.702" y2="5.842" width="0.8128" layer="16"/>
-<wire x1="28.702" y1="5.842" x2="27.178" y2="5.842" width="0.8128" layer="16"/>
-<wire x1="27.178" y1="5.842" x2="25.654" y2="7.366" width="0.8128" layer="16"/>
-<via x="25.654" y="7.366" extent="1-16" drill="0.6"/>
-<wire x1="22.86" y1="7.45" x2="25.57" y2="7.45" width="0.8128" layer="1"/>
-<wire x1="25.57" y1="7.45" x2="25.654" y2="7.366" width="0.8128" layer="1"/>
+<wire x1="33.02" y1="5.08" x2="29.21" y2="5.08" width="0.8128" layer="16"/>
+<wire x1="29.21" y1="5.08" x2="25.908" y2="8.382" width="0.8128" layer="16"/>
+<via x="25.908" y="8.382" extent="1-16" drill="0.6"/>
+<wire x1="22.86" y1="7.45" x2="24.468" y2="7.45" width="0.8128" layer="1"/>
+<wire x1="24.468" y1="7.45" x2="25.4" y2="8.382" width="0.8128" layer="1"/>
+<wire x1="25.4" y1="8.382" x2="25.908" y2="8.382" width="0.8128" layer="1"/>
 </signal>
 </signals>
-<errors>
-</errors>
 </board>
 </drawing>

Commit message: Pegelwandler mit FET
Parts:
- removed R5: 6.2k, resistor:R1206
- removed T1, T3: BC547, transistor:SOT23-EBC
- removed T2: BC557, transistor:SOT23-BCE
- added Q29, Q30: 2N7002P, transistor-small-signal:SOT23
- added Q31: BSS84, transistor-small-signal:SOT23
- R3: value 110k -> 100k
- R4: value NB -> 100k
- R7: value 7.5k -> 100k
- moved TP1 3.81 mm to (41.9, 5.08)
- moved R3 1.27 mm to (6.35, 6.35), flipped to the bottom, turned to 0 degrees
- moved R4 1.27 mm to (16.5, 3.81), turned to 90 degrees
- moved R7 1.27 mm to (6.35, 3.81)
Connections:
- removed net CP: IC1.13, IC1.8, IC2.13, IC2.8, IC3.13, IC3.8, IC4.13, IC4.8, Q1.2, Q10.2, Q11.2, Q12.2, Q13.2, Q14.2, Q15.2, Q16.2, Q17.2, Q18.2, Q19.2, Q2.2, Q20.2, Q21.2, Q22.2, Q23.2, Q24.2, Q25.1, Q25.3, Q26.1, Q26.3, Q27.1, Q27.3, Q28.1, Q28.3, Q3.2, Q4.2, Q5.2, Q6.2, Q7.2, Q8.2, Q9.2, R2.1, R6.1, R9.1, T1.E, T3.E, TP4.TP, U$1.20, U$2.P$4
- removed net N$33: R3.1, T1.B
- removed net N$35: R5.2, T2.B
- removed net N$36: R7.1, T3.B
- new net GND: IC1.13, IC1.8, IC2.13, IC2.8, IC3.13, IC3.8, IC4.13, IC4.8, Q1.2, Q10.2, Q11.2, Q12.2, Q13.2, Q14.2, Q15.2, Q16.2, Q17.2, Q18.2, Q19.2, Q2.2, Q20.2, Q21.2, Q22.2, Q23.2, Q24.2, Q25.1, Q25.3, Q26.1, Q26.3, Q27.1, Q27.3, Q28.1, Q28.3, Q29.2, Q3.2, Q30.2, Q4.2, Q5.2, Q6.2, Q7.2, Q8.2, Q9.2, R2.1, R3.1, R6.1, R7.1, R9.1, TP4.TP, U$1.20, U$2.P$4
- net +5V: now also Q31.2; no longer T2.E
- net N$34: now also Q30.3, Q31.1; no longer R5.1, T1.C
- net N$37: now also Q29.1
- net POWER_ON: now also Q29.3; no longer T3.C
- net TRIGGER: now also Q31.3; no longer T2.C
- net TRIGGER_UC: now also Q30.1
Routing:
- net GND: track 0.00 -> 339.2 mm, vias 0 -> 48
- net CP: track 327.9 -> 0.00 mm, vias 48 -> 0
- net N$37: track 2.39 -> 38.0 mm
- net N$36: track 35.3 -> 0.00 mm
- net TRIGGER_UC: track 2.39 -> 13.2 mm
- net N$35: track 5.76 -> 0.00 mm
- net N$34: track 7.18 -> 11.7 mm
- net +5V: track 97.1 -> 101.5 mm
- net N$33: track 3.81 -> 0.00 mm
- net POWER_ON: track 6.07 -> 4.51 mm
- added copper zone on layer 1, net GND
- added copper zone on layer 16, net GND
- removed copper zone on layer 1, net CP
- removed copper zone on layer 16, net CP
