File: hardware/e-wall-smd.sch (EAGLE design)
At the start: 66 parts, among them IC1 74HCT595D, IC2 74HCT595D, IC3 74HCT595D, IC4 74HCT595D, Q1 2N7002P, Q10 2N7002P, Q11 2N7002P, Q12 2N7002P, Q13 2N7002P, Q14 2N7002P, Q15 2N7002P, Q16 2N7002P, Q17 2N7002P, Q18 2N7002P, Q19 2N7002P, Q2 2N7002P, Q20 2N7002P, Q21 2N7002P, Q22 2N7002P, Q23 2N7002P, Q24 2N7002P, Q25 IRF8313P, Q26 IRF8313P, Q27 IRF8313P, Q28 IRF8313P, Q29 2N7002P, Q3 2N7002P, Q30 2N7002P, Q31 BSS84, Q4 2N7002P, Q5 2N7002P, Q6 2N7002P, Q7 2N7002P, Q8 2N7002P, Q9 2N7002P

Commit message: Transistortypen festgelegt
Parts:
- Q1, Q10, Q11, Q12, Q13, Q14, Q15, Q16, Q17, Q18, Q19, Q2, Q20, Q21, Q22, Q23, Q24, Q29, Q3, Q30, Q4, Q5, Q6, Q7, Q8, Q9: value 2N7002P -> SI2302CDS
- Q25, Q26, Q27, Q28: value IRF8313P -> SI4214DDY
- Q31: value BSS84 -> SI2347DS
Changed lines of the file:
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@@
 <part name="GND10" library="supply1" deviceset="GND" device=""/>
 <part name="U$1" library="msp430launchpad" deviceset="MSP430LAUNCHPAD_BASIC" device="" value="MSP430G2 Launchpad"/>
-<part name="Q1" library="transistor-small-signal" deviceset="BSS123" device="" value="2N7002P"/>
-<part name="Q2" library="transistor-small-signal" deviceset="BSS123" device="" value="2N7002P"/>
-<part name="Q3" library="transistor-small-signal" deviceset="BSS123" device="" value="2N7002P"/>
-<part name="Q4" library="transistor-small-signal" deviceset="BSS123" device="" value="2N7002P"/>
-<part name="Q5" library="transistor-small-signal" deviceset="BSS123" device="" value="2N7002P"/>
-<part name="Q6" library="transistor-small-signal" deviceset="BSS123" device="" value="2N7002P"/>
-<part name="Q7" library="transistor-small-signal" deviceset="BSS123" device="" value="2N7002P"/>
-<part name="Q8" library="transistor-small-signal" deviceset="BSS123" device="" value="2N7002P"/>
+<part name="Q1" library="transistor-small-signal" deviceset="BSS123" device="" value="SI2302CDS"/>
+<part name="Q2" library="transistor-small-signal" deviceset="BSS123" device="" value="SI2302CDS"/>
+<part name="Q3" library="transistor-small-signal" deviceset="BSS123" device="" value="SI2302CDS"/>
+<part name="Q4" library="transistor-small-signal" deviceset="BSS123" device="" value="SI2302CDS"/>
+<part name="Q5" library="transistor-small-signal" deviceset="BSS123" device="" value="SI2302CDS"/>
+<part name="Q6" library="transistor-small-signal" deviceset="BSS123" device="" value="SI2302CDS"/>
+<part name="Q7" library="transistor-small-signal" deviceset="BSS123" device="" value="SI2302CDS"/>
+<part name="Q8" library="transistor-small-signal" deviceset="BSS123" device="" value="SI2302CDS"/>
 <part name="GND4" library="supply1" deviceset="GND" device=""/>
 <part name="GND5" library="supply1" deviceset="GND" device=""/>
@@
 <part name="GND13" library="supply1" deviceset="GND" device=""/>
 <part name="GND14" library="supply1" deviceset="GND" device=""/>
-<part name="Q9" library="transistor-small-signal" deviceset="BSS123" device="" value="2N7002P"/>
-<part name="Q10" library="transistor-small-signal" deviceset="BSS123" device="" value="2N7002P"/>
-<part name="Q11" library="transistor-small-signal" deviceset="BSS123" device="" value="2N7002P"/>
-<part name="Q12" library="transistor-small-signal" deviceset="BSS123" device="" value="2N7002P"/>
-<part name="Q13" library="transistor-small-signal" deviceset="BSS123" device="" value="2N7002P"/>
-<part name="Q14" library="transistor-small-signal" deviceset="BSS123" device="" value="2N7002P"/>
-<part name="Q15" library="transistor-small-signal" deviceset="BSS123" device="" value="2N7002P"/>
-<part name="Q16" library="transistor-small-signal" deviceset="BSS123" device="" value="2N7002P"/>
+<part name="Q9" library="transistor-small-signal" deviceset="BSS123" device="" value="SI2302CDS"/>
+<part name="Q10" library="transistor-small-signal" deviceset="BSS123" device="" value="SI2302CDS"/>
+<part name="Q11" library="transistor-small-signal" deviceset="BSS123" device="" value="SI2302CDS"/>
+<part name="Q12" library="transistor-small-signal" deviceset="BSS123" device="" value="SI2302CDS"/>
+<part name="Q13" library="transistor-small-signal" deviceset="BSS123" device="" value="SI2302CDS"/>
+<part name="Q14" library="transistor-small-signal" deviceset="BSS123" device="" value="SI2302CDS"/>
+<part name="Q15" library="transistor-small-signal" deviceset="BSS123" device="" value="SI2302CDS"/>
+<part name="Q16" library="transistor-small-signal" deviceset="BSS123" device="" value="SI2302CDS"/>
 <part name="GND15" library="supply1" deviceset="GND" device=""/>
 <part name="GND16" library="supply1" deviceset="GND" device=""/>
@@
 <part name="GND21" library="supply1" deviceset="GND" device=""/>
 <part name="GND22" library="supply1" deviceset="GND" device=""/>
-<part name="Q17" library="transistor-small-signal" deviceset="BSS123" device="" value="2N7002P"/>
-<part name="Q18" library="transistor-small-signal" deviceset="BSS123" device="" value="2N7002P"/>
-<part name="Q19" library="transistor-small-signal" deviceset="BSS123" device="" value="2N7002P"/>
-<part name="Q20" library="transistor-small-signal" deviceset="BSS123" device="" value="2N7002P"/>
-<part name="Q21" library="transistor-small-signal" deviceset="BSS123" device="" value="2N7002P"/>
-<part name="Q22" library="transistor-small-signal" deviceset="BSS123" device="" value="2N7002P"/>
-<part name="Q23" library="transistor-small-signal" deviceset="BSS123" device="" value="2N7002P"/>
-<part name="Q24" library="transistor-small-signal" deviceset="BSS123" device="" value="2N7002P"/>
+<part name="Q17" library="transistor-small-signal" deviceset="BSS123" device="" value="SI2302CDS"/>
+<part name="Q18" library="transistor-small-signal" deviceset="BSS123" device="" value="SI2302CDS"/>
+<part name="Q19" library="transistor-small-signal" deviceset="BSS123" device="" value="SI2302CDS"/>
+<part name="Q20" library="transistor-small-signal" deviceset="BSS123" device="" value="SI2302CDS"/>
+<part name="Q21" library="transistor-small-signal" deviceset="BSS123" device="" value="SI2302CDS"/>
+<part name="Q22" library="transistor-small-signal" deviceset="BSS123" device="" value="SI2302CDS"/>
+<part name="Q23" library="transistor-small-signal" deviceset="BSS123" device="" value="SI2302CDS"/>
+<part name="Q24" library="transistor-small-signal" deviceset="BSS123" device="" value="SI2302CDS"/>
 <part name="GND23" library="supply1" deviceset="GND" device=""/>
 <part name="GND24" library="supply1" deviceset="GND" device=""/>
@@
 <part name="IC4" library="74xx-eu" deviceset="74*595" device="D" technology="HCT" value="74HCT595D"/>
 <part name="GND35" library="supply1" deviceset="GND" device=""/>
-<part name="Q25" library="transistor-power" deviceset="IRF8313P" device=""/>
-<part name="Q26" library="transistor-power" deviceset="IRF8313P" device=""/>
-<part name="Q27" library="transistor-power" deviceset="IRF8313P" device=""/>
-<part name="Q28" library="transistor-power" deviceset="IRF8313P" device=""/>
+<part name="Q25" library="transistor-power" deviceset="IRF8313P" device="" value="SI4214DDY"/>
+<part name="Q26" library="transistor-power" deviceset="IRF8313P" device="" value="SI4214DDY"/>
+<part name="Q27" library="transistor-power" deviceset="IRF8313P" device="" value="SI4214DDY"/>
+<part name="Q28" library="transistor-power" deviceset="IRF8313P" device="" value="SI4214DDY"/>
 <part name="GND36" library="supply1" deviceset="GND" device=""/>
 <part name="GND37" library="supply1" deviceset="GND" device=""/>
@@
 <part name="P+27" library="supply1" deviceset="+12V" device=""/>
 <part name="GND48" library="supply1" deviceset="GND" device=""/>
-<part name="Q29" library="transistor-small-signal" deviceset="BSS123" device="" value="2N7002P"/>
-<part name="Q30" library="transistor-small-signal" deviceset="BSS123" device="" value="2N7002P"/>
-<part name="Q31" library="transistor-small-signal" deviceset="BSS84" device=""/>
+<part name="Q29" library="transistor-small-signal" deviceset="BSS123" device="" value="SI2302CDS"/>
+<part name="Q30" library="transistor-small-signal" deviceset="BSS123" device="" value="SI2302CDS"/>
+<part name="Q31" library="transistor-small-signal" deviceset="BSS84" device="" value="SI2347DS"/>
 <part name="GND49" library="supply1" deviceset="GND" device=""/>
 <part name="GND50" library="supply1" deviceset="GND" device=""/>
